File: PCB/Relay board shield.brd (EAGLE design)
At the start: 74.6 x 80 mm, 13 parts, among them K1 RELAY-SPDT-JZC-11F, K10 RELAY-SPDT-JZC-11F, K11 RELAY-SPDT-JZC-11F, K2 RELAY-SPDT-JZC-11F, K3 RELAY-SPDT-JZC-11F, K4 RELAY-SPDT-JZC-11F, K5 RELAY-SPDT-JZC-11F, K6 RELAY-SPDT-JZC-11F, K7 RELAY-SPDT-JZC-11F, K8 RELAY-SPDT-JZC-11F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

Commit message: finished pcb
Parts:
- moved B1 6.35 mm to (29.2, 39.4)
- moved J2 6.35 mm to (66.0, 50.8)
- moved K11 6.35 mm to (47.0, 38.1)
- moved K2 6.35 mm to (12.7, 38.1)
- moved K5 6.35 mm to (24.1, 38.1)
- moved K8 6.35 mm to (35.6, 38.1)
- moved K3 6.35 mm to (12.7, 17.8)
- moved K6 6.35 mm to (24.1, 17.8)
- moved K9 6.35 mm to (35.6, 17.8)
- moved K1 6.35 mm to (12.7, 58.4)
- moved K10 6.35 mm to (47.0, 58.4)
- moved K4 6.35 mm to (24.1, 58.4)
- moved K7 6.35 mm to (35.6, 58.4)
Routing:
- net GND: track 0.00 -> 159.3 mm, vias 0 -> 1
- net RELAY10: track 0.00 -> 55.2 mm, vias 0 -> 1
- net RELAY3: track 0.00 -> 54.7 mm
- net RELAY6: track 0.00 -> 54.3 mm, vias 0 -> 1
- net RELAY9: track 0.00 -> 50.9 mm
- net RELAY8: track 0.00 -> 47.7 mm
- net RELAY11: track 0.00 -> 47.3 mm
- net RELAY5: track 0.00 -> 46.8 mm
Other:
- board size 74.6 x 80 mm -> 70.8 x 72.4 mm
- board text added: "1 2 3 4 5 6 7"
